Commit message: 完整上传 src/vrx 源码与东坡湖环境，编译产物移出仓库
- src/vrx：VRX 上游源码全量入库（此前因内嵌 .git 只记录了空指针，内容未上传）
- 新增东坡湖环境：worlds/dongpo_lake.sdf、models/dongpo_lake_terrain 等、
  tools/make_dongpo_terrain.py、launch/hu501.launch.py、卫星底图素材
- build/install/log 与 __pycache__ 移出跟踪并加入 .gitignore（本地 colcon build --merge-install 生成）
- README：编译命令改为 colcon build --merge-install（必需），移除失效的
  教程文档引用，图片引用更新为东坡湖截图

File: hu501urdf/urdf/hu501urdf.urdf.xacro (robot description, xacro)
@@ -41,11 +41,10 @@
       </material>
     </visual>
+    <!-- 碰撞用包围盒代替 STL 网格: 网格-高度场碰撞对在 dartsim/bullet 下
+         不可靠, 且盒碰撞更省算力 -->
     <collision>
-      <origin
-        xyz="-0.29592 -1.03178 -0.05518"
-        rpy="0 0 3.14159" />
-      <geometry>
-        <mesh
-          filename="package://hu501urdf/meshes/base_link.STL" />
+      <origin xyz="0 0 -0.05" rpy="0 0 0" />
+      <geometry>
+        <box size="1.04 0.52 0.4" />
       </geometry>
     </collision>
